Commit message: bbox envers

File: urdf/g500arm5e_uwsim.urdf (robot description, URDF)
Before this commit: robot g500arm5e, 8 links, 7 joints
Joints:
- joint Elbow: limit lower=-3.14159265359 upper=3.14159265359 effort=10 velocity=1 -> lower=0.314159265359 upper=1.57079632679 effort=10 velocity=1
- joint JawOpening: limit lower=-3.14159265359 upper=3.14159265359 effort=10 velocity=1 -> lower=0 upper=1.57079632679 effort=10 velocity=.5
- joint JawOpening2: limit lower=-3.14159265359 upper=3.14159265359 effort=10 velocity=1 -> lower=0 upper=1.57079632679 effort=10 velocity=.5
- joint JawRotate: limit lower=-3.14159265359 upper=3.14159265359 effort=10 velocity=1 -> lower=-1.57079632679 upper=1.57079632679 effort=10 velocity=1
- joint Shoulder: limit lower=-3.14159265359 upper=3.14159265359 effort=10 velocity=1 -> lower=0 upper=1.57079632679 effort=10 velocity=1
- joint Slew: limit lower=-3.14159265359 upper=3.14159265359 effort=10 velocity=1 -> lower=-1.57079632679 upper=1.57079632679 effort=10 velocity=1
