Commit message: debug path issue with meshes

File: urdf/bbox.xacro (robot description, xacro)
@@ -6,5 +6,5 @@
       <origin rpy="0 0 0" xyz="0 0 0"/>
       <geometry>
-          <mesh filename="package://freefloating_gazebo_demo/objects/blackbox_uib_trimesh.dae"/>
+          <mesh filename="file://$(env HOME)/.uwsim/data/objects/blackbox_uib_trimesh.dae"/>
       </geometry>
     </visual>
@@ -17,5 +17,5 @@
       <origin xyz="0 0 0" rpy="0 0 0"/>
      <geometry>
-          <mesh filename="package://freefloating_gazebo_demo/objects/blackbox_uib_trimesh.dae"/>
+          <mesh filename="file://$(env HOME)/.uwsim/data/objects/blackbox_uib_trimesh.dae"/>
       </geometry>
     </collision>

File: urdf/g500.xacro (robot description, xacro)
@@ -47,6 +47,4 @@
         <updateRate>100</updateRate>
         <link>base_link</link>
-        <bodyCommandTopic>body_command</bodyCommandTopic>
-        <jointCommandTopic>joint_command</jointCommandTopic>
         <!-- for each thruster, give the map to XYZ+RPY and the maximum effort -->
         <thruster>

Commit message: debug path to mesh

File: urdf/bbox.xacro (robot description, xacro)
@@ -6,5 +6,5 @@
       <origin rpy="0 0 0" xyz="0 0 0"/>
       <geometry>
-          <mesh filename="file://$(env HOME)/.uwsim/data/objects/blackbox_uib_trimesh.dae"/>
+          <mesh filename="package://freefloating_gazebo_demo/objects/blackbox_uib_trimesh.dae"/>
       </geometry>
     </visual>
@@ -17,5 +17,5 @@
       <origin xyz="0 0 0" rpy="0 0 0"/>
      <geometry>
-          <mesh filename="file://$(env HOME)/.uwsim/data/objects/blackbox_uib_trimesh.dae"/>
+          <mesh filename="package://freefloating_gazebo_demo/objects/blackbox_uib_trimesh.dae"/>
       </geometry>
     </collision>
