Commit message: PID control may be available even when using thruster force

File: urdf/steering_thrusters.xacro (robot description, xacro)
@@ -20,5 +20,5 @@
             <child link="${name}"/>
             <origin rpy="${rpy}" xyz="${xyz}"/>
-            <dynamics damping="10.0"/>
+            <dynamics damping="1.0"/>
             <axis xyz="0 1 0"/>
             <limit effort="30" velocity="5.0" lower="-${PI/2}" upper="${PI/2}" />
