Commit message: dummy joints in steering URDF to display wrenches in Rviz

File: urdf/steering_thrusters.urdf (robot description, URDF)
Before this commit: robot steering_auv, 3 links, 2 joints
Links:
- added link fwd_left_virt
- added link fwd_right_virt
Joints:
- added joint fwd_left_j: type revolute, parent base_link, child fwd_left, origin xyz=-0.5 0.18 0 rpy=0 1.57079632679 0, axis 0 1 0, limit lower=-1.57079632679 upper=1.57079632679 effort=30 velocity=5.0
- added joint fwd_right_j: type revolute, parent base_link, child fwd_right, origin xyz=-0.5 -0.18 0 rpy=0 1.57079632679 0, axis 0 1 0, limit lower=-1.57079632679 upper=1.57079632679 effort=30 velocity=5.0
- joint fwd_left: axis 0 1 0 -> 0 0 1; child fwd_left -> fwd_left_virt; origin xyz=-0.5 0.18 0 rpy=0 1.57079632679 0 -> (none); parent base_link -> fwd_left; type revolute -> prismatic
- joint fwd_right: axis 0 1 0 -> 0 0 1; child fwd_right -> fwd_right_virt; origin xyz=-0.5 -0.18 0 rpy=0 1.57079632679 0 -> (none); parent base_link -> fwd_right; type revolute -> prismatic

File: urdf/steering_thrusters.xacro (robot description, xacro)
@@ -20,5 +20,5 @@
             <child link="${name}"/>
             <origin rpy="${rpy}" xyz="${xyz}"/>
-            <dynamics damping="1.0"/>
+            <dynamics damping="10.0"/>
             <axis xyz="0 1 0"/>
             <limit effort="30" velocity="5.0" lower="-${PI/2}" upper="${PI/2}" />
@@ -119,3 +119,22 @@
     <xacro:thruster_link name="fwd_left" xyz="${-body_length/3} ${body_radius+tr2} 0" rpy="0 ${PI/2} 0"/>
     <xacro:thruster_link name="fwd_right" xyz="${-body_length/3} -${body_radius+tr2} 0" rpy="0 ${PI/2} 0"/>
+    <!-- Dummy links to display wrench in Rviz, autogenerated -->
+    <link name="thr2"/>
+    <joint name="thr2" type="fixed">
+        <parent link="base_link"/>
+        <child link="thr2"/>
+        <origin rpy="-1.57079632679 -0.0 0.0" xyz="0.0 0.0 0.0"/>
+    </joint>
+    <link name="thr3"/>
+    <joint name="thr3" type="fixed">
+        <parent link="base_link"/>
+        <child link="thr3"/>
+        <origin rpy="0.0 -0.0 0.0" xyz="-0.45 0.0 0.0"/>
+    </joint>
+    <link name="thr4"/>
+    <joint name="thr4" type="fixed">
+        <parent link="base_link"/>
+        <child link="thr4"/>
+        <origin rpy="0.0 -0.0 0.0" xyz="0.45 0.0 0.0"/>
+    </joint>
         </robot>
