Commit message: consistent with Z-thruster orientation

File: urdf/vectored.xacro (robot description, xacro)
@@ -35,5 +35,5 @@
             </visual>
             <visual name="${name}_2">
-                <origin xyz="0 0 -${(tl1+tl2)/2}"/>
+                <origin xyz="0 0 ${(tl1+tl2)/2}"/>
                 <geometry>
                     <cylinder length="${tl2}" radius="${tr2}"/>
@@ -75,6 +75,6 @@
                     <name>fwd_right</name>
                 </thruster>
-                <!--    these thrusters are fixed and the map can be hard-coded
-                        they will be given a name (thr2 to thr4)  -->
+                <!-- these thrusters are fixed and the map can be hard-coded
+                     they will be given a name (thr2 to thr4)  -->
                 <thruster>
                     <map>0 1 0 0 0 0</map>
@@ -117,24 +117,17 @@
             </link>
     <!-- Define two steering thrusters, with assume force control in Z-direction -->
-    <xacro:thruster_link name="fwd_left" xyz="${-body_length/3} ${body_radius+tr2} 0" rpy="0 ${PI/2} 0"/>
-    <xacro:thruster_link name="fwd_right" xyz="${-body_length/3} -${body_radius+tr2} 0" rpy="0 ${PI/2} 0"/>
+    <xacro:thruster_link name="fwd_left" xyz="${-body_length/3} ${body_radius+tr2} 0" rpy="0 ${-PI/2} 0"/>
+    <xacro:thruster_link name="fwd_right" xyz="${-body_length/3} -${body_radius+tr2} 0" rpy="0 ${-PI/2} 0"/>
+    <xacro:macro name="thruster_dummy_link" params="name xyz rpy">
+        <joint name="${name}" type="fixed">
+            <parent link="base_link"/>
+            <child link="${name}"/>
+            <origin rpy="${rpy}" xyz="${xyz}"/>
+        </joint>
+        <link name="${name}"/>
+    </xacro:macro>
     <!-- Dummy links to display wrench in Rviz, autogenerated -->
-    <link name="thr2"/>
-    <joint name="thr2" type="fixed">
-        <parent link="base_link"/>
-        <child link="thr2"/>
-        <origin rpy="-1.57079632679 -0.0 0.0" xyz="0.0 0.0 0.0"/>
-    </joint>
-    <link name="thr3"/>
-    <joint name="thr3" type="fixed">
-        <parent link="base_link"/>
-        <child link="thr3"/>
-        <origin rpy="0.0 -0.0 0.0" xyz="-0.45 0.0 0.0"/>
-    </joint>
-    <link name="thr4"/>
-    <joint name="thr4" type="fixed">
-        <parent link="base_link"/>
-        <child link="thr4"/>
-        <origin rpy="0.0 -0.0 0.0" xyz="0.45 0.0 0.0"/>
-    </joint>
+    <xacro:thruster_dummy_link name="thr2" xyz="0.0 0.0 0.0" rpy="1.57079632679 -0.0 0.0"/>
+    <xacro:thruster_dummy_link name="thr3" xyz="-0.45 0.0 0.0" rpy="0.0 -0.0 0.0"/>
+    <xacro:thruster_dummy_link name="thr4" xyz="0.45 0.0 0.0" rpy="0.0 -0.0 0.0"/>
         </robot>
