Commit message: removed occurences of old message BodySetpoint

File: urdf/g500_dummy.urdf (robot description, URDF)
Before this commit: robot body, 0 links, 5 joints
Joints:
- joint x: limit lower=-10 upper=10 -> lower=-17 upper=23
- joint y: limit lower=-10.0 upper=10.0 -> lower=-13.5 upper=26.6
- joint z: limit lower=-12.0 upper=0.0 -> lower=-20.0 upper=0.0

File: urdf/vectored.xacro (robot description, xacro)
@@ -113,5 +113,5 @@
                     <origin xyz= "0 0 0"/>
                     <limit radius="${body_radius}"/>
-                    <damping xyz="6 100 100" rpy="20 50 50"/>
+                    <damping xyz="40 100 100" rpy="20 50 50"/>
                 </buoyancy>
             </link>
