Commit message: demo en cours

File: urdf/arm5e.xacro (robot description, xacro)
@@ -139,5 +139,5 @@
     <axis xyz="0 -1 0"/>
     <origin rpy="0 0 0" xyz="0.07 0 0.04"/>
-    <dynamics damping="0.8"/>
+    <dynamics damping="0.3"/>
     <limit lower="0" upper="${PI/2}" velocity=".5" effort="10"/>
     </joint>
@@ -157,5 +157,5 @@
     <axis xyz="0 1 0"/>
     <origin rpy="0 0 0" xyz="0.07 0 -0.04"/>
-    <dynamics damping="0.8"/>
+    <dynamics damping="0.3"/>
     <limit lower="0" upper="${PI/2}" velocity=".5" effort="10"/>
     </joint>

File: urdf/bbox.xacro (robot description, xacro)
@@ -22,4 +22,5 @@
     <buoyancy>
     <compensation>0</compensation>
+    <damping xyz="0 0 0"/>
     </buoyancy>
   </link>

Commit message: demo 3 dof

File: urdf/arm5e.xacro (robot description, xacro)
@@ -68,5 +68,5 @@
     <origin rpy="0 0 0" xyz="0 0 0"/>
     <dynamics damping="0.8"/>
-    <limit lower="${-PI/2}" upper="${PI/2}" velocity="1" effort="10"/>
+    <limit lower="${-PI/2}" upper="${PI/2}" velocity="1" effort="500"/>
   </joint>
  <link name="part2">
@@ -86,5 +86,5 @@
     <origin rpy="0 0.209 0" xyz="0.077 0 -0.130"/>
     <dynamics damping="0.8"/>
-    <limit lower="0" upper="${PI/2}" velocity="1" effort="10"/>
+    <limit lower="0" upper="${PI/2}" velocity="1" effort="500"/>
   </joint>
  <link name="part3">
@@ -104,5 +104,5 @@
     <origin rpy=" 0 0.262 0 " xyz="0.44278 0 0"/>
     <dynamics damping="0.8"/>
-    <limit lower="${PI/10}" upper="${PI/2}" velocity="1" effort="10"/>
+    <limit lower="${PI/10}" upper="${PI/2}" velocity="1" effort="500"/>
     </joint>
   <link name="part4_base">
@@ -116,5 +116,5 @@
     <buoyancy><compensation>1.0</compensation></buoyancy>
   </link>
-  <joint name="JawRotate" type="revolute">
+  <!--<joint name="JawRotate" type="revolute">
     <parent link="part3"/>
     <child link="part4_base"/>
@@ -122,6 +122,74 @@
     <origin rpy="0 0 0" xyz="0.320 0 0.077 "/>
     <dynamics damping="0.8"/>
-    <limit lower="${-PI/2}" upper="${PI/2}" velocity="1" effort="10"/>
-    </joint>
+    <limit lower="${-PI/2}" upper="${PI/2}" velocity="1" effort="200"/>
+    </joint>-->
+    <joint name="JawRotate" type="fixed">
+    <parent link="part3"/>
+    <child link="part4_base"/>
+    <axis xyz="1 0 0"/>
+    <origin rpy="0 0 0" xyz="0.320 0 0.077 "/>
+    </joint>
+    <link name="part5">
+    <visual>
+      <origin rpy="0 0 0" xyz="0 0 0"/>
+       <geometry>
+        <cylinder length="0.08" radius="0.01"/>
+      </geometry>
+      <material name="orange"/>
+    </visual>
+       <collision>
+      <origin rpy="0 0 0" xyz="0 0 0"/>
+       <geometry>
+        <cylinder length="0.08" radius="0.01"/>
+      </geometry>
+    </collision>
+    <xacro:cyl_inertial mass=".05" radius=".01" length=".06" />
+    </link>
+    <joint name="part4_to_5" type="fixed">
+    <parent link="part4_base"/>
+    <child link="part5"/>
+    <origin rpy="0 1.57079632679 0" xyz=".12 0 0 "/>
+    </joint>
+    <link name="part6">
+    <visual>
+      <origin rpy="0 0 0" xyz="0 0 .03"/>
+       <geometry>
+        <cylinder length="0.06" radius="0.008"/>
+      </geometry>
+    </visual>
+    <collision>
+      <origin rpy="0 0 0" xyz="0 0 .03"/>
+       <geometry>
+        <cylinder length="0.06" radius="0.008"/>
+      </geometry>
+    </collision>
+    <xacro:cyl_inertial mass=".05" radius=".01" length=".06" />
+    </link>
+    <joint name="part5_to_6" type="fixed">
+    <parent link="part5"/>
+    <child link="part6"/>
+    <origin xyz="0 .0 .035 " rpy="0 .6 0"/>
+    </joint>
+    <link name="part7">
+    <visual>
+      <origin rpy="0 0 0" xyz="0 0 .03"/>
+       <geometry>
+        <cylinder length="0.06" radius="0.006"/>
+      </geometry>
+    </visual>
+    <collision>
+      <origin rpy="0 0 0" xyz="0 0 .03"/>
+       <geometry>
+        <cylinder length="0.06" radius="0.006"/>
+      </geometry>
+    </collision>
+    <xacro:cyl_inertial mass=".05" radius=".01" length=".06" />
+    </link>
+    <joint name="part6_to_7" type="fixed">
+    <parent link="part6"/>
+    <child link="part7"/>
+    <origin xyz="0 .0 .06 " rpy="0 .6 0"/>
+    </joint>
+<!--
   <link name="part4_jaw1">
     <visual>
@@ -145,6 +213,6 @@
     <axis xyz="0 -1 0"/>
     <origin rpy="0 0 0" xyz="0.07 0 0.04"/>
-    <dynamics damping="0.3"/>
-    <limit lower="0" upper="${PI/2}" velocity=".5" effort="10"/>
+    <dynamics damping="0.8"/>
+    <limit lower="-.01" upper="${PI/2}" velocity=".1" effort="100"/>
     </joint>
 <link name="part4_jaw2">
@@ -169,6 +237,6 @@
     <axis xyz="0 1 0"/>
     <origin rpy="0 0 0" xyz="0.07 0 -0.04"/>
-    <dynamics damping="0.3"/>
-    <limit lower="0" upper="${PI/2}" velocity=".5" effort="10"/>
-    </joint>
+    <dynamics damping="0.8"/>
+    <limit lower="-.01" upper="${PI/2}" velocity=".1" effort="100"/>
+    </joint>-->
 </robot>

File: urdf/bbox.xacro (robot description, xacro)
@@ -11,5 +11,5 @@
     <inertial>
       <origin rpy="0 0 0" xyz="0 0 0"/>
-      <mass value="8.0"/>
+      <mass value="4.0"/>
       <inertia ixx="1" ixy="0.0" ixz="0.0" iyy="1" iyz="0" izz="1"/>
     </inertial>

File: urdf/g500arm5e_uwsim.urdf (robot description, URDF)
Before this commit: robot g500arm5e, 8 links, 7 joints
Links:
- removed link part4_jaw1
- removed link part4_jaw2
- added link part5; visual cylinder length=0.08 radius=0.01
- added link part6; visual cylinder length=0.06 radius=0.008
- added link part7; visual cylinder length=0.06 radius=0.006
Joints:
- removed joint JawOpening
- removed joint JawOpening2
- added joint part4_to_5: type fixed, parent part4_base, child part5, origin xyz=.12 0 0  rpy=0 1.57079632679 0
- added joint part5_to_6: type fixed, parent part5, child part6, origin xyz=0 .0 .035  rpy=0 .6 0
- added joint part6_to_7: type fixed, parent part6, child part7, origin xyz=0 .0 .06  rpy=0 .6 0
- joint JawRotate: limit lower=-1.57079632679 upper=1.57079632679 effort=10 velocity=1 -> (none); type revolute -> fixed

Commit message: add 4th joint in g500_arm5e demo

File: urdf/arm5e.xacro (robot description, xacro)
@@ -5,5 +5,5 @@
   <xacro:property name="arm_mass" value="1"/>
   <xacro:property name="arm_radius" value="0.10"/>
-  <xacro:property name="jaw_mass" value="0.1"/>
+  <xacro:property name="jaw_mass" value="0.5"/>
   <xacro:property name="jaw_radius" value="0.05"/>
   <xacro:property name="eps" value="0.00000001"/>
@@ -116,5 +116,5 @@
     <buoyancy><compensation>1.0</compensation></buoyancy>
   </link>
-  <!--<joint name="JawRotate" type="revolute">
+  <joint name="JawRotate" type="revolute">
     <parent link="part3"/>
     <child link="part4_base"/>
@@ -123,11 +123,11 @@
     <dynamics damping="0.8"/>
     <limit lower="${-PI/2}" upper="${PI/2}" velocity="1" effort="200"/>
-    </joint>-->
-    <joint name="JawRotate" type="fixed">
+    </joint>
+    <!--<joint name="JawRotate" type="fixed">
     <parent link="part3"/>
     <child link="part4_base"/>
     <axis xyz="1 0 0"/>
     <origin rpy="0 0 0" xyz="0.320 0 0.077 "/>
-    </joint>
+    </joint>-->
     <link name="part5">
     <visual>
@@ -138,5 +138,5 @@
       <material name="orange"/>
     </visual>
-       <collision>
+   <collision>
       <origin rpy="0 0 0" xyz="0 0 0"/>
        <geometry>
@@ -145,4 +145,5 @@
     </collision>
     <xacro:cyl_inertial mass=".05" radius=".01" length=".06" />
+    <buoyancy><compensation>1.0</compensation></buoyancy>
     </link>
     <joint name="part4_to_5" type="fixed">
@@ -165,4 +166,5 @@
     </collision>
     <xacro:cyl_inertial mass=".05" radius=".01" length=".06" />
+    <buoyancy><compensation>1.0</compensation></buoyancy>
     </link>
     <joint name="part5_to_6" type="fixed">
@@ -184,5 +186,6 @@
       </geometry>
     </collision>
-    <xacro:cyl_inertial mass=".05" radius=".01" length=".06" />
+    <xacro:cyl_inertial mass=".1" radius=".01" length=".06" />
+    <buoyancy><compensation>1.0</compensation></buoyancy>
     </link>
     <joint name="part6_to_7" type="fixed">
