Commit message: update readme.md

File: urdf/g500.xacro (robot description, xacro)
@@ -45,28 +45,29 @@
     <plugin name="freefloating_gazebo_control" filename="libfreefloating_gazebo_control.so">
         <switchService>switch</switchService>
-            <link>base_link</link>
-            <bodyCommandTopic>body_command</bodyCommandTopic>
-            <jointCommandTopic>joint_command</jointCommandTopic>
-            <!-- for each thruster, give the map to XYZ+RPY and the maximum effort -->
-            <thruster>
-                <map>-1 0 0 0 0 ${-body_width/2}</map>
-                <effort>30</effort>
-            </thruster>
-            <thruster>
-                <map>-1 0 0 0 0 ${body_width/2}</map>
-                <effort>30</effort>
-            </thruster>
-            <thruster>
-                <map>0 1 0 0 0 0</map>
-                <effort>30</effort>
-            </thruster>
-            <thruster>
-                <map>0 0 -1 0 0 0</map>
-                <effort>30</effort>
-            </thruster>
-            <thruster>
-                <map>0 0 -1 0 ${-2*X_cog} 0</map>
-                <effort>30</effort>
-            </thruster>
+        <updateRate>100</updateRate>
+        <link>base_link</link>
+        <bodyCommandTopic>body_command</bodyCommandTopic>
+        <jointCommandTopic>joint_command</jointCommandTopic>
+        <!-- for each thruster, give the map to XYZ+RPY and the maximum effort -->
+        <thruster>
+            <map>-1 0 0 0 0 ${-body_width/2}</map>
+            <effort>30</effort>
+        </thruster>
+        <thruster>
+            <map>-1 0 0 0 0 ${body_width/2}</map>
+            <effort>30</effort>
+        </thruster>
+        <thruster>
+            <map>0 1 0 0 0 0</map>
+            <effort>30</effort>
+        </thruster>
+        <thruster>
+            <map>0 0 -1 0 0 0</map>
+            <effort>30</effort>
+        </thruster>
+        <thruster>
+            <map>0 0 -1 0 ${-2*X_cog} 0</map>
+            <effort>30</effort>
+        </thruster>
     </plugin>
     </gazebo>
@@ -99,5 +100,5 @@
       <origin xyz= "${X_cog} 0 ${body_height*body_bottom_mass/(2*body_top_mass+body_bottom_mass)/2}"/>
       <limit radius=".5"/>
-      <damping xyz="40 80 80"/>
+      <damping xyz="60 100 100"/>
   </buoyancy>
   </link>

File: urdf/g500arm5e_uwsim.urdf (robot description, URDF)
Before this commit: robot g500arm5e, 9 links, 8 joints
Joints:
- joint Elbow: limit lower=0.314159265359 upper=1.57079632679 effort=10 velocity=1 -> lower=0.314159265359 upper=1.57079632679 effort=500 velocity=1
- joint Shoulder: limit lower=0 upper=1.57079632679 effort=10 velocity=1 -> lower=0 upper=1.57079632679 effort=500 velocity=1
- joint Slew: limit lower=-1.57079632679 upper=1.57079632679 effort=10 velocity=1 -> lower=-1.57079632679 upper=1.57079632679 effort=500 velocity=1

Commit message: consistent with latest ffg

File: urdf/g500.xacro (robot description, xacro)
@@ -94,10 +94,15 @@
       </geometry>
     </collision-->
-  <buoyancy>
-      <compensation>1.01</compensation>
-      <origin xyz= "${X_cog} 0 ${body_height*body_bottom_mass/(2*body_top_mass+body_bottom_mass)/2}"/>
-      <limit radius=".5"/>
-      <damping xyz="60 100 100" rpy="20 50 50"/>
-  </buoyancy>
+    <fluid>
+        <density>1</density>
+        <origin xyz= "${X_cog} 0 ${body_height*body_bottom_mass/(2*body_top_mass+body_bottom_mass)/2}"/>
+        <buoyancy>
+            <compensation>1.01</compensation>
+            <limit radius="0.5"/>
+        </buoyancy>
+        <hydrodynamics>
+            <drag xyz="60 100 100" rpy="20 50 50" type="linear"/>
+        </hydrodynamics>
+    </fluid>
   </link>
 </robot>
